Commit message: working minitaur controlled

File: fast_adaptation_embedding/fast_adaptation_embedding/env/assets/pybullet_data/old_quadruped/minitaur.urdf (robot description, URDF)
Before this commit: robot quadruped, 31 links, 30 joints
Links:
- removed link contact_back_leftR_link
- removed link contact_back_rightL_link
- removed link contact_front_leftR_link
- removed link contact_front_rightL_link
- link motor_front_leftR_link: geometry visual mesh filename=tmotor3.obj scale=1 1 1
Joints:
- removed joint contact_back_leftR
- removed joint contact_back_rightL
- removed joint contact_front_leftR
- removed joint contact_front_rightL
- joint knee_back_leftL_link: type continuous -> revolute
- joint knee_back_leftR_link: type continuous -> revolute
- joint knee_back_rightL_link: type continuous -> revolute
- joint knee_back_rightR_link: type continuous -> revolute
- joint knee_front_leftL_link: type continuous -> revolute
- joint knee_front_leftR_link: type continuous -> revolute
- joint knee_front_rightL_link: type continuous -> revolute
- joint knee_front_rightR_link: type continuous -> revolute
