Commit message: increase of the stadium size

File: fast_adaptation_embedding/fast_adaptation_embedding/env/assets/pybullet_data/plane.urdf (robot description, URDF)
Before this commit: robot plane, 1 links, 0 joints
Links:
- link planeLink: geometry collision box size=100 100 10; visual mesh filename=plane.obj scale=1 1 1
