Commit message: correct feet position

File: fast_adaptation_embedding/fast_adaptation_embedding/env/assets/pybullet_data/quadruped/minitaur.urdf (robot description, URDF)
Before this commit: robot quadruped, 31 links, 30 joints
Joints:
- joint contact_back_leftR: parent lower_leg_back_leftR_link -> lower_leg_back_leftL_link
- joint contact_back_rightL: parent lower_leg_back_rightL_link -> lower_leg_back_rightR_link
- joint contact_front_leftR: parent lower_leg_front_leftR_link -> lower_leg_front_leftL_link
- joint contact_front_rightL: parent lower_leg_front_rightL_link -> lower_leg_front_rightR_link
